File: gemschematic.sch (EAGLE design)
At the start: 57 parts, among them J1 USB, J3 QWIIC, J5 U.FL, Q1 2N3904, Q2 BSS138, Q3 MBT3904DW1T1, U1 ESP-WROOM-32NARROW, U2 AP2112K-3.3, U3 3.3V, U4 RFM96W, U5 CH340C, U6 BMP180, X1 GPS_PA1010D

Commit message: PCB 2/10/22
Parts:
- removed STM32L496ZG-P: STM32F733ZET6, STM32F733ZET6:STM32F733ZET6
- added U7: STM32L073RZT6, STM32L073RZT6:STM32L073RZT6
- JP5: device adafruit:PINHD-1X1 -> pinhead:PINHD-1X2
Connections:
- removed net ADC1_IN8: STM32L496ZG-P.PC5
- removed net ADC3_IN12: STM32L496ZG-P.PF9
- removed net GPIO: STM32L496ZG-P.PC1
- removed net GPIO1: STM32L496ZG-P.PA0
- removed net I2C2_SCL: STM32L496ZG-P.PF1
- removed net I2C2_SDA: STM32L496ZG-P.PF0
- removed net SPI1: STM32L496ZG-P.PA1
- removed net UART1: STM32L496ZG-P.PA2
- removed net UART2: STM32L496ZG-P.PA3
- new net DHT22: U7.PC1
- new net PHOTO: U7.PC0
- new net SOIL: U7.PC3
- new net TEMP: U7.PC2
- new net USART_RX: U7.PA3
- new net USART_TX: U7.PA2
- net 3.3V: now also U7.VDDA
- net GND: now also U7.VSSA
- net MISO: now also U7.PC12; no longer STM32L496ZG-P.PA6
- net MOSI: now also U7.PC11; no longer STM32L496ZG-P.PA7
- net SCK: now also U7.PC10
- net SCL: now also U7.PB7
- net SDA: now also U7.PB6
- net VCC: no longer STM32L496ZG-P.VDD
Changed lines of the file:
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@@
 </classes>
 <parts>
-<part name="STM32L496ZG-P" library="STM32F733ZET6" deviceset="STM32F733ZET6" device=""/>
 <part name="DHT22" library="con-molex" library_urn="urn:adsk.eagle:library:165" deviceset="22-23-2041" device="" package3d_urn="urn:adsk.eagle:package:8078635/1"/>
 <part name="PULLUP" library="adafruit" library_urn="urn:adsk.eagle:library:420" deviceset="R-US_" device="0204/2V" package3d_urn="urn:adsk.eagle:package:6240630/1" value="10k">
@@
 <part name="U6" library="BMP180" deviceset="BMP180" device=""/>
 <part name="GND24" library="supply1" library_urn="urn:adsk.eagle:library:371" deviceset="GND" device=""/>
-<part name="JP5" library="adafruit" library_urn="urn:adsk.eagle:library:420" deviceset="PINHD-1X1" device="" package3d_urn="urn:adsk.eagle:package:6240654/1"/>
+<part name="JP5" library="pinhead" library_urn="urn:adsk.eagle:library:325" deviceset="PINHD-1X2" device="" package3d_urn="urn:adsk.eagle:package:22435/2"/>
+<part name="U7" library="STM32L073RZT6" deviceset="STM32L073RZT6" device=""/>
 </parts>
 <sheets>
@@
 <text x="-53.34" y="223.52" size="1.778" layer="91">Probe Circuit (Soil)</text>
 <text x="-45.72" y="119.38" size="1.778" layer="91">Temp/Humid Header Pins</text>
-<text x="30.48" y="162.56" size="1.778" layer="91">Microcontroller</text>
+<text x="55.88" y="160.02" size="1.778" layer="91">Microcontroller</text>
 <text x="185.42" y="43.18" size="1.778" layer="91">G</text>
 <text x="190.5" y="35.56" size="1.778" layer="91">S</text>
@@
 </plain>
 <instances>
-<instance part="STM32L496ZG-P" gate="G$1" x="58.42" y="48.26" smashed="yes">
-<attribute name="NAME" x="30.48" y="156.21" size="1.778" layer="95"/>
-</instance>
 <instance part="DHT22" gate="-1" x="-20.32" y="109.22" smashed="yes">
 <attribute name="NAME" x="-17.78" y="108.458" size="1.524" layer="95"/>
@@
 <attribute name="VALUE" x="205.74" y="-53.34" size="1.778" layer="96" rot="R90"/>
 </instance>
-<instance part="JP5" gate="G$1" x="-129.54" y="109.22" smashed="yes">
-<attribute name="NAME" x="-135.89" y="112.395" size="1.778" layer="95"/>
-<attribute name="VALUE" x="-135.89" y="104.14" size="1.778" layer="96"/>
+<instance part="JP5" gate="G$1" x="-132.08" y="106.68" smashed="yes">
+<attribute name="NAME" x="-138.43" y="112.395" size="1.778" layer="95"/>
+<attribute name="VALUE" x="-138.43" y="101.6" size="1.778" layer="96"/>
+</instance>
+<instance part="U7" gate="G$1" x="71.12" y="83.82" smashed="yes">
+<attribute name="NAME" x="50.8" y="143.24" size="2.0828" layer="95" ratio="10" rot="SR0"/>
+<attribute name="VALUE" x="50.8" y="21.4" size="2.0828" layer="96" ratio="10" rot="SR0"/>
 </instance>
 </instances>
@@
 <wire x1="-71.12" y1="111.76" x2="-78.74" y2="111.76" width="0.1524" layer="91"/>
 <label x="-78.74" y="111.76" size="1.778" layer="95"/>
-</segment>
-<segment>
-<pinref part="STM32L496ZG-P" gate="G$1" pin="VDD"/>
-<wire x1="91.44" y1="149.86" x2="99.06" y2="149.86" width="0.1524" layer="91"/>
-<label x="99.06" y="149.86" size="1.778" layer="95"/>
 </segment>
 </net>
@@
 <pinref part="GND24" gate="1" pin="GND"/>
 </segment>
+<segment>
+<pinref part="U7" gate="G$1" pin="VSSA"/>
+<wire x1="96.52" y1="30.48" x2="114.3" y2="30.48" width="0.1524" layer="91"/>
+<label x="111.76" y="30.48" size="1.778" layer="95"/>
+</segment>
 </net>
 <net name="SIG" class="0">
@@
 <wire x1="-162.56" y1="-78.74" x2="-162.56" y2="-81.28" width="0.1524" layer="91"/>
 </segment>
+<segment>
+<pinref part="U7" gate="G$1" pin="VDDA"/>
+<wire x1="96.52" y1="137.16" x2="111.76" y2="137.16" width="0.1524" layer="91"/>
+<label x="106.68" y="137.16" size="1.778" layer="95"/>
+</segment>
 </net>
 <net name="1PPS" class="0">
@@
 <label x="-2.54" y="-91.44" size="1.27" layer="95" xref="yes"/>
 </segment>
+<segment>
+<pinref part="U7" gate="G$1" pin="PB7"/>
+<wire x1="45.72" y1="55.88" x2="30.48" y2="55.88" width="0.1524" layer="91"/>
+<label x="30.48" y="55.88" size="1.778" layer="95"/>
+</segment>
 </net>
 <net name="SDA" class="0">
@@
 <wire x1="-5.08" y1="-93.98" x2="-2.54" y2="-93.98" width="0.1524" layer="91"/>
 <label x="-2.54" y="-93.98" size="1.27" layer="95" xref="yes"/>
+</segment>
+<segment>
+<pinref part="U7" gate="G$1" pin="PB6"/>
+<wire x1="45.72" y1="58.42" x2="30.48" y2="58.42" width="0.1524" layer="91"/>
+<label x="30.48" y="58.42" size="1.778" layer="95"/>
 </segment>
 </net>
@@
 </segment>
 <segment>
-<pinref part="STM32L496ZG-P" gate="G$1" pin="PA6"/>
-<wire x1="25.4" y1="104.14" x2="15.24" y2="104.14" width="0.1524" layer="91"/>
-<label x="15.24" y="104.14" size="1.778" layer="95"/>
+<pinref part="U7" gate="G$1" pin="PC12"/>
+<wire x1="96.52" y1="86.36" x2="111.76" y2="86.36" width="0.1524" layer="91"/>
+<label x="106.68" y="86.36" size="1.778" layer="95"/>
 </segment>
 </net>
@@
 </segment>
 <segment>
-<pinref part="STM32L496ZG-P" gate="G$1" pin="PA7"/>
-<wire x1="25.4" y1="101.6" x2="15.24" y2="101.6" width="0.1524" layer="91"/>
-<label x="15.24" y="101.6" size="1.778" layer="95"/>
+<pinref part="U7" gate="G$1" pin="PC11"/>
+<wire x1="96.52" y1="88.9" x2="111.76" y2="88.9" width="0.1524" layer="91"/>
+<label x="106.68" y="88.9" size="1.778" layer="95"/>
 </segment>
 </net>
@@
 <label x="-93.98" y="25.4" size="1.27" layer="95" xref="yes"/>
 <pinref part="U4" gate="G$1" pin="SCK"/>
+</segment>
+<segment>
+<pinref part="U7" gate="G$1" pin="PC10"/>
+<wire x1="96.52" y1="91.44" x2="111.76" y2="91.44" width="0.1524" layer="91"/>
+<label x="106.68" y="91.44" size="1.778" layer="95"/>
 </segment>
 </net>
@@
 </segment>
 </net>
-<net name="GPIO1" class="0">
-<segment>
-<pinref part="STM32L496ZG-P" gate="G$1" pin="PA0"/>
-<wire x1="25.4" y1="119.38" x2="15.24" y2="119.38" width="0.1524" layer="91"/>
-<label x="15.24" y="119.38" size="1.778" layer="95"/>
-</segment>
-</net>
-<net name="SPI1" class="0">
-<segment>
-<pinref part="STM32L496ZG-P" gate="G$1" pin="PA1"/>
-<wire x1="25.4" y1="116.84" x2="15.24" y2="116.84" width="0.1524" layer="91"/>
-<label x="15.24" y="116.84" size="1.778" layer="95"/>
-</segment>
-</net>
-<net name="ADC3_IN12" class="0">
-<segment>
-<pinref part="STM32L496ZG-P" gate="G$1" pin="PF9"/>
-<wire x1="91.44" y1="53.34" x2="101.6" y2="53.34" width="0.1524" layer="91"/>
-<label x="101.6" y="53.34" size="1.778" layer="95"/>
-</segment>
-</net>
-<net name="I2C2_SDA" class="0">
-<segment>
-<pinref part="STM32L496ZG-P" gate="G$1" pin="PF0"/>
-<wire x1="91.44" y1="76.2" x2="101.6" y2="76.2" width="0.1524" layer="91"/>
-<label x="101.6" y="76.2" size="1.778" layer="95"/>
-</segment>
-</net>
-<net name="I2C2_SCL" class="0">
-<segment>
-<pinref part="STM32L496ZG-P" gate="G$1" pin="PF1"/>
-<wire x1="91.44" y1="73.66" x2="101.6" y2="73.66" width="0.1524" layer="91"/>
-<label x="101.6" y="73.66" size="1.778" layer="95"/>
-</segment>
-</net>
-<net name="ADC1_IN8" class="0">
-<segment>
-<pinref part="STM32L496ZG-P" gate="G$1" pin="PC5"/>
-<wire x1="25.4" y1="20.32" x2="15.24" y2="20.32" width="0.1524" layer="91"/>
-<label x="10.16" y="20.32" size="1.778" layer="95"/>
-</segment>
-</net>
-<net name="UART1" class="0">
-<segment>
-<pinref part="STM32L496ZG-P" gate="G$1" pin="PA2"/>
-<wire x1="25.4" y1="114.3" x2="15.24" y2="114.3" width="0.1524" layer="91"/>
-<label x="15.24" y="114.3" size="1.778" layer="95"/>
-</segment>
-</net>
-<net name="UART2" class="0">
-<segment>
-<pinref part="STM32L496ZG-P" gate="G$1" pin="PA3"/>
-<wire x1="25.4" y1="111.76" x2="15.24" y2="111.76" width="0.1524" layer="91"/>
-<label x="15.24" y="111.76" size="1.778" layer="95"/>
-</segment>
-</net>
-<net name="GPIO" class="0">
-<segment>
-<pinref part="STM32L496ZG-P" gate="G$1" pin="PC1"/>
-<wire x1="25.4" y1="30.48" x2="17.78" y2="30.48" width="0.1524" layer="91"/>
-<label x="15.24" y="30.48" size="1.778" layer="95"/>
-</segment>
-</net>
 <net name="PF0" class="0">
 <segment>
@@
 <segment>
 <pinref part="JP5" gate="G$1" pin="1"/>
-<wire x1="-132.08" y1="109.22" x2="-144.78" y2="109.22" width="0.1524" layer="91"/>
+<wire x1="-134.62" y1="109.22" x2="-144.78" y2="109.22" width="0.1524" layer="91"/>
 <label x="-144.78" y="109.22" size="1.778" layer="95"/>
 </segment>
 </net>
+<net name="USART_TX" class="0">
+<segment>
+<pinref part="U7" gate="G$1" pin="PA2"/>
+<wire x1="45.72" y1="111.76" x2="30.48" y2="111.76" width="0.1524" layer="91"/>
+<label x="30.48" y="111.76" size="1.778" layer="95"/>
+</segment>
+</net>
+<net name="USART_RX" class="0">
+<segment>
+<pinref part="U7" gate="G$1" pin="PA3"/>
+<wire x1="45.72" y1="109.22" x2="30.48" y2="109.22" width="0.1524" layer="91"/>
+<label x="30.48" y="109.22" size="1.778" layer="95"/>
+</segment>
+</net>
+<net name="PHOTO" class="0">
+<segment>
+<pinref part="U7" gate="G$1" pin="PC0"/>
+<wire x1="96.52" y1="116.84" x2="111.76" y2="116.84" width="0.1524" layer="91"/>
+<label x="104.14" y="116.84" size="1.778" layer="95"/>
+</segment>
+</net>
+<net name="DHT22" class="0">
+<segment>
+<pinref part="U7" gate="G$1" pin="PC1"/>
+<wire x1="96.52" y1="114.3" x2="111.76" y2="114.3" width="0.1524" layer="91"/>
+<label x="104.14" y="114.3" size="1.778" layer="95"/>
+</segment>
+</net>
+<net name="TEMP" class="0">
+<segment>
+<pinref part="U7" gate="G$1" pin="PC2"/>
+<wire x1="96.52" y1="111.76" x2="111.76" y2="111.76" width="0.1524" layer="91"/>
+<label x="104.14" y="111.76" size="1.778" layer="95"/>
+</segment>
+</net>
+<net name="SOIL" class="0">
+<segment>
+<pinref part="U7" gate="G$1" pin="PC3"/>
+<wire x1="96.52" y1="109.22" x2="111.76" y2="109.22" width="0.1524" layer="91"/>
+<label x="106.68" y="109.22" size="1.778" layer="95"/>
+</segment>
+</net>

Commit message: Add files via upload
Parts:
- removed B1: (no value), microbuilder:BATTERYCR1220_2
- removed C1: 0.1uF, microbuilder:CAP_CERAMIC0603_NO
- removed C2, C3: 10uF, microbuilder:CAP_CERAMIC0805-NOOUTLINE
- removed C4: 10uF, SparkFun-Capacitors:10UF-0603-6.3V-20%
- removed C5, C6: 0.1uF, SparkFun-Capacitors:0.1UF-0603-25V-(+80/-20%)
- removed C7, C8: 1.0uF, SparkFun-Capacitors:1.0UF-0603-16V-10%
- removed C9: 4.7uF, SparkFun-Capacitors:4.7UF-0603-6.3V-(10%)
- removed CONN3, CONN4: STEMMA_I2C_QT, microbuilder:STEMMA_I2C_QT
- removed D1: GREEN, microbuilder:LED0603_NOOUTLINE
- removed D2: 1N4148, microbuilder:DIODESOD-323
- removed D3: RED, microbuilder:LED0603_NOOUTLINE
- removed D4: RED, SparkFun-LED:LED-RED0603
- removed D5: GREEN, SparkFun-LED:LED-GREEN0603
- removed FB1: FERRITE, microbuilder:FERRITE-0805NO
- removed J1: USB, SparkFun-Connectors:USB_MICRO-B_HALF_PTH_MILL
- removed J3: QWIIC, SparkFun-Connectors:QWIIC_CONNECTORJS-1MM
- removed J4: (no value), SparkFun-Connectors:CONN_08NO_SILK_FEMALE_PTH
- removed J5: U.FL, SparkFun-Connectors:U.FL
- removed J8: (no value), SparkFun-Connectors:CONN_01PTH_NO_SILK_YES_STOP
- removed J9: (no value), SparkFun-Connectors:CONN_10NO_SILK_PTH_FEMALE
- removed JP1: DNP, SparkFun-Connectors:M03POLAR
- removed JP2: (no value), SparkFun-Connectors:M03SCREW_LOCK
- removed JP3, JP4: (no value), microbuilder:HEADER-1X670MIL
- removed JP5: (no value), pinhead:PINHD-1X2
- removed PULLUP: 10k, adafruit:R-US_0204/2V
- removed Q1: 2N3904, SparkFun-DiscreteSemi:TRANSISTOR_NPNMMBT2222A
- removed Q2: BSS138, microbuilder:MOSFET-N_DUAL
- removed Q3: MBT3904DW1T1, esp32-thing-temp:MBT3904DW1T1
- removed R10, R17, R18, R6, R8: 10k, SparkFun-Resistors:10KOHM-0603-1/10W-1%
- removed R2: 100, SparkFun-Resistors:100OHM-1/4W-5%(0603)
- removed R3, R4, R5: 10K, microbuilder:RESISTOR_4PACK
- removed R7, R9: 1k, SparkFun-Resistors:1KOHM-0603-1/10W-1%
- removed S1: RESET, SparkFun-Switches:MOMENTARY-SWITCH-SPST-2-SMD-4.6X2.8MM
- removed S2: 0, SparkFun-Switches:MOMENTARY-SWITCH-SPST-2-SMD-4.6X2.8MM
- removed U1: ESP-WROOM-32NARROW, esp32_lora_gateway:ESP-WROOM-32NARROW
- removed U2: AP2112K-3.3, microbuilder:VREG_SOT23-5
- removed U3: 3.3V, SparkFun-IC-Power:V_REG_AP2112K-3.3V
- removed U4: RFM96W, SparkX:RFM96W
- removed U5: CH340C, SparkFun-IC-Comms:CH340C
- removed U6: BMP180, BMP180:BMP180
- removed X1: GPS_PA1010D, microbuilder:GPS_PA1010D
- added BARO: 22-23-2041, con-molex:22-23-2041
- added BLUETOOTH: 87438-06, con-molex:87438-06
- added GPS1JUMPER, GPS2JUMPER: (no value), microbuilder:HEADER-1X670MIL
- added LDRJUMPER: (no value), pinhead:PINHD-1X2
- added LORA1JUMPER: (no value), SparkFun-Connectors:CONN_08NO_SILK_FEMALE_PTH
- added LORA2JUMPER: (no value), SparkFun-Connectors:CONN_10NO_SILK_PTH_FEMALE
- added LORANT: (no value), SparkFun-Connectors:CONN_01PTH_NO_SILK_YES_STOP
- added PULLUP1, PULLUP2: 4.7k, adafruit:R-US_0204/2V
- added SOILJUMPER: (no value), SparkFun-Connectors:M03SCREW_LOCK
- DS18B20: value 22-23-2041 -> (none); device con-molex:22-23-2041 -> adafruit:PINHD-1X3
- R1: value 10k -> 270; device SparkFun-Resistors:100OHM-1/4W-5%(0603) -> adafruit:R-US_0204/2V
Connections:
- removed net !DTR: Q3Q2.E, R17.1, U5.!DTR
- removed net !RTS: Q3Q1.E, R18.1, U5.!RTS
- removed net 0: Q3Q2.C, R10.1, S2.3, S2.4, U1.IO0
- removed net D+: J1.D+, U5.UD+
- removed net D-: J1.D-, U5.UD-
- removed net DATA: DHT22-2.S, DS18B20-2.S, PULLUP.1
- removed net DHT22: U7.PC1
- removed net IO17: R9.1, U1.IO17
- removed net MISO: J4.2, U1.MISO_H/IO12, U4.MISO, U7.PC12
- removed net MOSI: J4.1, U1.MOSI_HIO13, U4.MOSI, U7.PC11
- removed net N$10: Q3Q1.B, R17.2
- removed net N$12: Q3Q2.B, R18.2
- removed net N$2: D1.C, R4G$3.2
- removed net N$3: D3.C, R4G$1.2, R4G$2.2
- removed net N$4: D4.C, R7.2
- removed net N$5: D5.A, R9.2
- removed net OUT: FB1.P$1, U2.OUT
- removed net PC5: JP5.1
- removed net PF0: U6.SDA
- removed net PF1: U6.SCL
- removed net PHOTO: U7.PC0
- removed net PROBE1: Q1.B
- removed net PROBE2: R2.1
- removed net RFM_CS: U1.IO16, U4.NSS
- removed net RFM_DIO1/33: U1.XTAL_N/IO33, U4.DIO1
- removed net RFM_DIO2/32: U1.XTAL_P/IO32, U4.DIO2
- removed net RFM_INT/26: U1.IO26, U4.DIO0
- removed net RFM_RST: R8.1, U4.!RESET
- removed net RXI_3V: D2.A, R3G$4.2, X1.RX
- removed net SCK: J4.3, U1.SCK_HIO14, U4.SCK, U7.PC10
- removed net SCL_3V: Q21.S, R5G$2.2, X1.SCL
- removed net SDA_3V: Q22.S, R5G$4.2, X1.SDA
- removed net SHIELD: J1.SHIELD
- removed net SIG: JP1.3, JP2.1, Q1.E, R1.2
- removed net SOIL: U7.PC3
- removed net TEMP: U7.PC2
- removed net USART_RX: U7.PA3
- removed net USART_TX: U7.PA2
- removed net VBACKUP: B1.+, X1.VBACKUP
- removed net VDDIO: U6.VDDIO
- removed net V_USB: C7.1, J1.VBUS, U3.EN, U3.IN
- new net BTRX: BLUETOOTH-2.S, U7.PC10
- new net BTTX: BLUETOOTH-3.S, U7.PA1
- new net GPSRX: GPS2JUMPER.4, U7.PA9
- new net GPSTX: GPS2JUMPER.5, U7.PA10
- new net MISOLORA: LORA1JUMPER.2, U7.PC12
- new net MOSILORA: LORA1JUMPER.1, U7.PC11
- new net PA0LDR: LDRJUMPER.1, R1.2, U7.PA0
- new net PC1DHT: DHT22-2.S, PULLUP1.1, U7.PC1
- new net PC2DS18B20: DS18B20.2, PULLUP2.1, U7.PC2
- new net PC3SOIL: SOILJUMPER.1, U7.PC3
- new net SCKLORA: LORA1JUMPER.3, U7.PC6
- new net SCLBARO: BARO-3.S, U7.PB6
- new net SDABARO: BARO-4.S, U7.PB7
- new net VIN: BARO-1.S
- net !RESET: now also GPS1JUMPER.6; no longer JP3.6, X1.!RESET
- net 1PPS: now also GPS2JUMPER.2; no longer D3.A, JP4.2, X1.PPS
- net 3.3V: now also GPS1JUMPER.2; no longer C1.1, C3.1, C4.1, C5.1, C8.1, C9.1, D1.A, D4.A, FB1.P$2, J3.2, J4.7, JP3.2, Q21.G, Q22.G, R10.2, R3G$4.1, R5G$2.1, R5G$4.1, R6.2, R8.2, U1.3V3, U3.OUT, U4.3.3V, U5.V3, U5.VCC, U7.VDDA, X1.VCC
- net ANT: now also LORANT.1; no longer J5.SIGNAL, J8.1, U4.ANT
- net GND: now also BARO-2.S, BLUETOOTH-5.S, DS18B20.3, GPS1JUMPER.3, GPS2JUMPER.1, LORA1JUMPER.8, LORA2JUMPER.10, SOILJUMPER.2; no longer B1.-, C1.2, C2.2, C3.2, C4.2, C5.2, C6.2, C7.2, C8.2, C9.2, CONN3G$1.GND, CONN4G$1.GND, D5.C, DS18B20-4.S, J1.GND, J3.1, J4.8, J5.GND@0, J5.GND@1, J9.10, JP1.2, JP2.2, JP3.3, JP4.1, R4G$1.1, R4G$2.1, R4G$3.1, R7.1, S1.1, S1.2, S2.1, S2.2, U1.GND, U1.GND@1, U1.GND@15, U1.GND@38, U2.GND, U3.GND, U4.GND, U5.GND, U6.GND, X1.GND
- net IO18: now also LORA2JUMPER.5; no longer J9.5, U1.SCK_V/IO18
- net IO19: now also LORA2JUMPER.6; no longer J9.6, U1.MISO_V/IO19
- net IO23: now also LORA2JUMPER.7; no longer J9.7, U1.MOSI_V/IO23
- net IO25: now also LORA1JUMPER.5; no longer J4.5, U1.IO25
- net IO27: now also LORA1JUMPER.4; no longer J4.4, U1.IO27
- net IO4: now also LORA2JUMPER.3; no longer J9.3, U1.IO4
- net IO5: now also LORA2JUMPER.4; no longer J9.4, U1.CS0_V/IO5
- net RESET: now also LORA1JUMPER.6; no longer C6.1, J4.6, Q3Q1.C, R6.1, S1.3, S1.4, U1.EN
- net RXI: now also LORA2JUMPER.8; no longer D2.C, J9.8, JP4.4, U1.RXD, U5.TXO
- net SCL: now also LORA2JUMPER.2; no longer CONN3G$1.SCL, CONN4G$1.SCL, J3.4, J9.2, JP3.4, Q21.D, R5G$1.2, U1.IO22, U7.PB7
- net SDA: now also LORA2JUMPER.1; no longer CONN3G$1.SDA, CONN4G$1.SDA, J3.3, J9.1, JP3.5, Q22.D, R5G$3.2, U1.IO21, U7.PB6
- net TXO: now also LORA2JUMPER.9; no longer J9.9, JP4.5, U1.TXD, U5.RXI, X1.TX
- net VCC: now also BLUETOOTH-4.S, DS18B20.1, GPS1JUMPER.1, GPS2JUMPER.3, LDRJUMPER.2, LORA1JUMPER.7, PULLUP1.2, PULLUP2.2, SOILJUMPER.3, U7.VDDA; no longer C2.1, CONN3G$1.V+, CONN4G$1.V+, DS18B20-1.S, JP1.1, JP2.3, JP3.1, JP4.3, PULLUP.2, Q1.C, R2.2, R5G$1.1, R5G$3.1, U2.EN, U2.IN
- net VDD: now also U7.VDD; no longer U6.VDD
- net WAKEUP: now also GPS2JUMPER.6; no longer JP4.6, X1.WAKEUP
Other:
- note added: "Bluetooth Jumpers"
- note added: "version 3"
- note removed: "600mA out 6V max in"
- note removed: "Auto Reset (LoRa)"
- note removed: "D"
- note removed: "ESP32-WROOM (LoRa)"
- note removed: "G"
- note removed: "GPS Main"
- note removed: "I2C Headers (GPS)"
- note removed: "I2C Pullups and Shift (GPS)"
- note removed: "LED and Buttons (LoRa)"
- note removed: "ON LED (GPS)"
- note removed: "Power Supply (GPS)"
- note removed: "Probe Circuit (Soil)"
- note removed: "RFM95HW (LoRa)"
- note removed: "S"
- note removed: "USB to Serial (LoRa)"
- note removed: "Voltage Regulator (LoRa)"
- moved on the sheet: DHT22-1, DHT22-2, DHT22-3, DHT22-4, R1
